Commit message: modifying xacro

File: install/robot_description/share/robot_description/urdf/xacro_variables.xacro (robot description, xacro)
@@ -5,10 +5,10 @@
   <!--Chasis_box-->
   <xacro:property name="chasis_box_length" value="0.478" />
-  <xacro:property name="chasis_box_width" value="0.28" />
-  <xacro:property name="chasis_box_height" value="0.05" />
+  <xacro:property name="chasis_box_width" value="0.3" />
+  <xacro:property name="chasis_box_height" value="0.15" />
   <!--Chasis_caster-->
-  <xacro:property name="chasis_caster_radius" value="0.0375" />
+  <xacro:property name="chasis_caster_radius" value="0.05" />
   <!--Wheel_cylinder-->
-  <xacro:property name="wheel_cylinder_radius" value="0.085" />
+  <xacro:property name="wheel_cylinder_radius" value="0.17" />
   <xacro:property name="wheel_cylinder_height" value="0.045" />
 <!--Positions-->
@@ -21,13 +21,13 @@
   <xacro:property name="chasis_box_ya" value="0" />
   <!--Chasis_caster-->
-  <xacro:property name="chasis_caster_x" value="-0.2" />
+  <xacro:property name="chasis_caster_x" value="-0.15" />
   <xacro:property name="chasis_caster_y" value="0" />
-  <xacro:property name="chasis_caster_z" value="-0.047" />
+  <xacro:property name="chasis_caster_z" value="-0.05" />
   <xacro:property name="chasis_caster_r" value="0" />
   <xacro:property name="chasis_caster_p" value="0" />
   <xacro:property name="chasis_caster_ya" value="0" />
-  <xacro:property name="chasis_caster2_x" value="0.2" />
+  <xacro:property name="chasis_caster2_x" value="0.15" />
   <xacro:property name="chasis_caster2_y" value="0" />
-  <xacro:property name="chasis_caster2_z" value="-0.047" />
+  <xacro:property name="chasis_caster2_z" value="-0.05" />
   <xacro:property name="chasis_caster2_r" value="0" />
   <xacro:property name="chasis_caster2_p" value="0" />

File: skyfood_ws/install/robot_description/share/robot_description/urdf/robot_base.xacro (robot description, xacro)
@@ -95,5 +95,5 @@
   <link name="lidar_link">
     <visual name="lidar_visual">
-      <origin xyz="0 0 0.07" rpy="0 0 0"/>
+      <origin xyz="0 0 0.01" rpy="0 0 0"/>
       <geometry>
         <cylinder radius="0.1" length="0.05"/>
@@ -104,9 +104,9 @@
     <parent link="chassis"/>
     <child link="lidar_link"/>
-    <origin xyz="0 0 0.07" rpy="0 0 0"/>
+    <origin xyz="0 0 0.24" rpy="0 0 0"/>
   </joint>
   <link name="camera_link">
     <visual name="camera_visual">
-      <origin xyz="0.11 0 0" rpy="0 0 0"/>
+      <origin xyz="0.01 0 0" rpy="0 0 0"/>
       <geometry>
         <box size="0.02 0.15 0.1"/>
@@ -117,5 +117,5 @@
     <parent link="chassis"/>
     <child link="camera_link"/>
-    <origin xyz="0.11 0 0" rpy="0 0 0"/>
+    <origin xyz="0.20 0 0" rpy="0 0 0"/>
   </joint>
   <!-- Include wheel and caster macros -->

File: skyfood_ws/install/robot_description/share/robot_description/urdf/xacro_variables.xacro (robot description, xacro)
@@ -4,12 +4,12 @@
 <!--Dimentions-->
   <!--Chasis_box-->
-  <xacro:property name="chasis_box_length" value="0.4" />
-  <xacro:property name="chasis_box_width" value="0.3" />
-  <xacro:property name="chasis_box_height" value="0.15" />
+  <xacro:property name="chasis_box_length" value="0.478" />
+  <xacro:property name="chasis_box_width" value="0.28" />
+  <xacro:property name="chasis_box_height" value="0.05" />
   <!--Chasis_caster-->
-  <xacro:property name="chasis_caster_radius" value="0.05" />
+  <xacro:property name="chasis_caster_radius" value="0.0375" />
   <!--Wheel_cylinder-->
-  <xacro:property name="wheel_cylinder_radius" value="0.1" />
-  <xacro:property name="wheel_cylinder_height" value="0.05" />
+  <xacro:property name="wheel_cylinder_radius" value="0.085" />
+  <xacro:property name="wheel_cylinder_height" value="0.045" />
 <!--Positions-->
   <!--Chasis_box-->
@@ -21,13 +21,13 @@
   <xacro:property name="chasis_box_ya" value="0" />
   <!--Chasis_caster-->
-  <xacro:property name="chasis_caster_x" value="-0.15" />
+  <xacro:property name="chasis_caster_x" value="-0.2" />
   <xacro:property name="chasis_caster_y" value="0" />
-  <xacro:property name="chasis_caster_z" value="-0.05" />
+  <xacro:property name="chasis_caster_z" value="-0.047" />
   <xacro:property name="chasis_caster_r" value="0" />
   <xacro:property name="chasis_caster_p" value="0" />
   <xacro:property name="chasis_caster_ya" value="0" />
-  <xacro:property name="chasis_caster2_x" value="0.15" />
+  <xacro:property name="chasis_caster2_x" value="0.2" />
   <xacro:property name="chasis_caster2_y" value="0" />
-  <xacro:property name="chasis_caster2_z" value="-0.05" />
+  <xacro:property name="chasis_caster2_z" value="-0.047" />
   <xacro:property name="chasis_caster2_r" value="0" />
   <xacro:property name="chasis_caster2_p" value="0" />
@@ -42,8 +42,8 @@
 <!--Joint variables-->
   <xacro:property name="right_wheel_x" value="0.0" />
-  <xacro:property name="right_wheel_y" value="0.20" />
+  <xacro:property name="right_wheel_y" value="0.166" />
   <xacro:property name="right_wheel_z" value="0" />
   <xacro:property name="left_wheel_x" value="0" />
-  <xacro:property name="left_wheel_y" value="-0.20" />
+  <xacro:property name="left_wheel_y" value="-0.166" />
   <xacro:property name="left_wheel_z" value="0" />
 </robot>
