Commit message: tower box

File: skyfood_ws/install/robot_description/share/robot_description/urdf/materials.xacro (robot description, xacro)
@@ -14,8 +14,8 @@
   </material>
   <material name="orange">
-    <color rgba="${255/255} ${108/255} ${10/255} 1.0"/>
+    <color rgba="1.0 0.4235 0.0392 1.0"/>
   </material>
   <material name="brown">
-    <color rgba="${222/255} ${207/255} ${195/255} 1.0"/>
+    <color rgba="0.8627 0.8157 0.7725 1.0"/>
   </material>
   <material name="red">

File: skyfood_ws/install/robot_description/share/robot_description/urdf/robot_base.xacro (robot description, xacro)
@@ -31,4 +31,17 @@
       <geometry>
         <box size="${chasis_box_length} ${chasis_box_width} ${chasis_box_height}"/>
+      </geometry>
+      <material name="red"/>
+    </visual>
+    <collision name='tower_collision'>
+      <origin xyz="0 0 0.58" rpy="0 0 0"/>
+      <geometry>
+        <box size="${tower_box_length} ${tower_box_width} ${tower_box_height}"/>
+      </geometry>
+    </collision>
+    <visual name='tower_visual'>
+      <origin xyz="0 0 0.58" rpy="0 0 0"/>
+      <geometry>
+        <box size="${tower_box_length} ${tower_box_width} ${tower_box_height}"/>
       </geometry>
       <material name="red"/>
@@ -78,5 +91,5 @@
         <sphere radius="${chasis_caster_radius}"/>
       </geometry>
-      <material name="orange"/>
+      <material name="red"/>
     </visual>
   </link>
@@ -97,5 +110,5 @@
       <origin xyz="0 0 0.01" rpy="0 0 0"/>
       <geometry>
-        <cylinder radius="0.1" length="0.05"/>
+        <cylinder radius="0.05" length="0.035"/>
       </geometry>
     </visual>
@@ -104,9 +117,9 @@
     <parent link="chassis"/>
     <child link="lidar_link"/>
-    <origin xyz="0 0 0.24" rpy="0 0 0"/>
+    <origin xyz="0 0 0.2" rpy="0 0 0"/>
   </joint>
   <link name="camera_link">
     <visual name="camera_visual">
-      <origin xyz="0.01 0 0" rpy="0 0 0"/>
+      <origin xyz="0 0 0" rpy="0 0 0"/>
       <geometry>
         <box size="0.02 0.15 0.1"/>
@@ -117,5 +130,5 @@
     <parent link="chassis"/>
     <child link="camera_link"/>
-    <origin xyz="0.20 0 0" rpy="0 0 0"/>
+    <origin xyz="0.239 0 0.84" rpy="0 0 0"/>
   </joint>
   <!-- Include wheel and caster macros -->

File: skyfood_ws/install/robot_description/share/robot_description/urdf/xacro_variables.xacro (robot description, xacro)
@@ -12,4 +12,8 @@
   <xacro:property name="wheel_cylinder_radius" value="0.085" />
   <xacro:property name="wheel_cylinder_height" value="0.045" />
+  <!--Tower box-->
+  <xacro:property name="tower_box_length" value="0.478" />
+  <xacro:property name="tower_box_width" value="0.448" />
+  <xacro:property name="tower_box_height" value="0.64" />
 <!--Positions-->
   <!--Chasis_box-->

File: skyfood_ws/src/robot_description/urdf/robot_base.xacro (robot description, xacro)
@@ -31,4 +31,17 @@
       <geometry>
         <box size="${chasis_box_length} ${chasis_box_width} ${chasis_box_height}"/>
+      </geometry>
+      <material name="red"/>
+    </visual>
+    <collision name='tower_collision'>
+      <origin xyz="0 0 0.58" rpy="0 0 0"/>
+      <geometry>
+        <box size="${tower_box_length} ${tower_box_width} ${tower_box_height}"/>
+      </geometry>
+    </collision>
+    <visual name='tower_visual'>
+      <origin xyz="0 0 0.58" rpy="0 0 0"/>
+      <geometry>
+        <box size="${tower_box_length} ${tower_box_width} ${tower_box_height}"/>
       </geometry>
       <material name="red"/>
@@ -97,5 +110,5 @@
       <origin xyz="0 0 0.01" rpy="0 0 0"/>
       <geometry>
-        <cylinder radius="0.1" length="0.05"/>
+        <cylinder radius="0.05" length="0.035"/>
       </geometry>
     </visual>
@@ -104,9 +117,9 @@
     <parent link="chassis"/>
     <child link="lidar_link"/>
-    <origin xyz="0 0 0.24" rpy="0 0 0"/>
+    <origin xyz="0 0 0.2" rpy="0 0 0"/>
   </joint>
   <link name="camera_link">
     <visual name="camera_visual">
-      <origin xyz="0.01 0 0" rpy="0 0 0"/>
+      <origin xyz="0 0 0" rpy="0 0 0"/>
       <geometry>
         <box size="0.02 0.15 0.1"/>
@@ -117,5 +130,5 @@
     <parent link="chassis"/>
     <child link="camera_link"/>
-    <origin xyz="0.20 0 0" rpy="0 0 0"/>
+    <origin xyz="0.239 0 0.84" rpy="0 0 0"/>
   </joint>
   <!-- Include wheel and caster macros -->
