Commit message: four caster, fix mass and friction

File: skyfood_ws/install/robot_description/share/robot_description/urdf/caster_ball.xacro (robot description, xacro)
@@ -26,5 +26,5 @@
     </visual>
     <collision name='caster_collision2'>
-      <origin xyz="${chasis_caster2_x} ${chasis_caster2_y} ${chasis_caster2_z}" rpy=" ${chasis_caster2_r} ${chasis_caster2_p} ${chasis_caster2_ya}"/>
+      <origin xyz="${chasis_caster2_x} ${chasis_caster2_y} ${chasis_caster2_z}" rpy=" ${chasis_caster_r} ${chasis_caster_p} ${chasis_caster_ya}"/>
       <geometry>
         <sphere radius="${chasis_caster_radius}"/>
@@ -42,5 +42,5 @@
     </collision>
     <visual name='caster2_visual'>
-      <origin xyz="${chasis_caster2_x} ${chasis_caster2_y} ${chasis_caster2_z}" rpy=" ${chasis_caster2_r} ${chasis_caster2_p} ${chasis_caster2_ya}"/>
+      <origin xyz="${chasis_caster2_x} ${chasis_caster2_y} ${chasis_caster2_z}" rpy=" ${chasis_caster_r} ${chasis_caster_p} ${chasis_caster_ya}"/>
       <geometry>
         <sphere radius="${chasis_caster_radius}"/>
@@ -49,3 +49,49 @@
     </visual>
   </xacro:macro>
+  <collision name='caster_collision3'>
+    <origin xyz="${chasis_caster3_x} ${chasis_caster3_y} ${chasis_caster3_z}" rpy=" ${chasis_caster_r} ${chasis_caster_p} ${chasis_caster_ya}"/>
+    <geometry>
+      <sphere radius="${chasis_caster_radius}"/>
+    </geometry>
+    <surface>
+      <friction>
+        <ode>
+          <mu>0</mu>
+          <mu2>0</mu2>
+          <slip1>1.0</slip1>
+          <slip2>1.0</slip2>
+        </ode>
+      </friction>
+    </surface>
+  </collision>
+  <visual name='caster3_visual'>
+    <origin xyz="${chasis_caster3_x} ${chasis_caster3_y} ${chasis_caster3_z}" rpy=" ${chasis_caster_r} ${chasis_caster_p} ${chasis_caster_ya}"/>
+    <geometry>
+      <sphere radius="${chasis_caster_radius}"/>
+    </geometry>
+    <material name="orange"/>
+  </visual>
+  <collision name='caster_collision4'>
+    <origin xyz="${chasis_caster4_x} ${chasis_caster4_y} ${chasis_caster4_z}" rpy=" ${chasis_caster_r} ${chasis_caster_p} ${chasis_caster_ya}"/>
+    <geometry>
+      <sphere radius="${chasis_caster_radius}"/>
+    </geometry>
+    <surface>
+      <friction>
+        <ode>
+          <mu>0</mu>
+          <mu2>0</mu2>
+          <slip1>1.0</slip1>
+          <slip2>1.0</slip2>
+        </ode>
+      </friction>
+    </surface>
+  </collision>
+  <visual name='caster4_visual'>
+    <origin xyz="${chasis_caster4_x} ${chasis_caster4_y} ${chasis_caster4_z}" rpy=" ${chasis_caster_r} ${chasis_caster_p} ${chasis_caster_ya}"/>
+    <geometry>
+      <sphere radius="${chasis_caster_radius}"/>
+    </geometry>
+    <material name="orange"/>
+  </visual>
 </robot>

File: skyfood_ws/install/robot_description/share/robot_description/urdf/robot_base.xacro (robot description, xacro)
@@ -13,7 +13,7 @@
     <pose>0 0 0.1 0 0 0</pose>
     <inertial>
-      <mass value="10.0"/>
+      <mass value="30.0"/>
       <origin xyz="0.0 0 0.1" rpy=" 0 0 0"/>
-      <box_inertia m="10" l="${chasis_box_length}" w="${chasis_box_width}" h="${chasis_box_height}"/>
+      <box_inertia m="30" l="${chasis_box_length}" w="${chasis_box_width}" h="${chasis_box_height}"/>
       <inertia
           ixx="0.5" ixy="0" ixz="0"
@@ -71,5 +71,5 @@
     </visual>
     <collision name='caster_collision2'>
-      <origin xyz="${chasis_caster2_x} ${chasis_caster2_y} ${chasis_caster2_z}" rpy=" ${chasis_caster2_r} ${chasis_caster2_p} ${chasis_caster2_ya}"/>
+      <origin xyz="${chasis_caster2_x} ${chasis_caster2_y} ${chasis_caster2_z}" rpy=" ${chasis_caster_r} ${chasis_caster_p} ${chasis_caster_ya}"/>
       <geometry>
         <sphere radius="${chasis_caster_radius}"/>
@@ -87,9 +87,55 @@
     </collision>
     <visual name='caster2_visual'>
-      <origin xyz="${chasis_caster2_x} ${chasis_caster2_y} ${chasis_caster2_z}" rpy=" ${chasis_caster2_r} ${chasis_caster2_p} ${chasis_caster2_ya}"/>
+      <origin xyz="${chasis_caster2_x} ${chasis_caster2_y} ${chasis_caster2_z}" rpy=" ${chasis_caster_r} ${chasis_caster_p} ${chasis_caster_ya}"/>
       <geometry>
         <sphere radius="${chasis_caster_radius}"/>
       </geometry>
-      <material name="red"/>
+      <material name="orange"/>
+    </visual>
+    <collision name='caster_collision3'>
+      <origin xyz="${chasis_caster3_x} ${chasis_caster3_y} ${chasis_caster3_z}" rpy=" ${chasis_caster_r} ${chasis_caster_p} ${chasis_caster_ya}"/>
+      <geometry>
+        <sphere radius="${chasis_caster_radius}"/>
+      </geometry>
+      <surface>
+        <friction>
+          <ode>
+            <mu>0</mu>
+            <mu2>0</mu2>
+            <slip1>1.0</slip1>
+            <slip2>1.0</slip2>
+          </ode>
+        </friction>
+      </surface>
+    </collision>
+    <visual name='caster3_visual'>
+      <origin xyz="${chasis_caster3_x} ${chasis_caster3_y} ${chasis_caster3_z}" rpy=" ${chasis_caster_r} ${chasis_caster_p} ${chasis_caster_ya}"/>
+      <geometry>
+        <sphere radius="${chasis_caster_radius}"/>
+      </geometry>
+      <material name="orange"/>
+    </visual>
+    <collision name='caster_collision4'>
+      <origin xyz="${chasis_caster4_x} ${chasis_caster4_y} ${chasis_caster4_z}" rpy=" ${chasis_caster_r} ${chasis_caster_p} ${chasis_caster_ya}"/>
+      <geometry>
+        <sphere radius="${chasis_caster_radius}"/>
+      </geometry>
+      <surface>
+        <friction>
+          <ode>
+            <mu>0</mu>
+            <mu2>0</mu2>
+            <slip1>1.0</slip1>
+            <slip2>1.0</slip2>
+          </ode>
+        </friction>
+      </surface>
+    </collision>
+    <visual name='caster4_visual'>
+      <origin xyz="${chasis_caster4_x} ${chasis_caster4_y} ${chasis_caster4_z}" rpy=" ${chasis_caster_r} ${chasis_caster_p} ${chasis_caster_ya}"/>
+      <geometry>
+        <sphere radius="${chasis_caster_radius}"/>
+      </geometry>
+      <material name="orange"/>
     </visual>
   </link>
@@ -117,5 +163,5 @@
     <parent link="chassis"/>
     <child link="lidar_link"/>
-    <origin xyz="0 0 0.2" rpy="0 0 0"/>
+    <origin xyz="0 0 0.18" rpy="0 0 0"/>
   </joint>
   <link name="camera_link">

File: skyfood_ws/install/robot_description/share/robot_description/urdf/wheels.xacro (robot description, xacro)
@@ -8,4 +8,12 @@
           <cylinder radius="${wheel_cylinder_radius}" length="${wheel_cylinder_height}"/>
         </geometry>
+        <surface>
+          <friction>
+            <ode>
+              <mu>1</mu>
+              <mu2>1</mu2>
+            </ode>
+          </friction>
+        </surface>
       </collision>
       <visual name="left_wheel_visual">
@@ -18,6 +26,6 @@
       <inertial>
         <origin xyz="${wheel_x} ${wheel_y} ${wheel_z}" rpy="${wheel_r} ${wheel_p} ${wheel_ya}"/>
-        <mass value="5"/>
-        <cylinder_inertia m="5" r="${wheel_cylinder_radius}" h="${wheel_cylinder_height}"/>
+        <mass value="1"/>
+        <cylinder_inertia m="1" r="${wheel_cylinder_radius}" h="${wheel_cylinder_height}"/>
         <inertia
           ixx="1.0" ixy="0.0" ixz="0.0"
@@ -32,4 +40,12 @@
           <cylinder radius="${wheel_cylinder_radius}" length="${wheel_cylinder_height}"/>
         </geometry>
+        <surface>
+          <friction>
+            <ode>
+              <mu>1</mu>
+              <mu2>1</mu2>
+            </ode>
+          </friction>
+        </surface>
       </collision>
       <visual name="right_wheel_visual">
@@ -42,6 +58,6 @@
       <inertial>
         <origin xyz="${wheel_x} ${wheel_y} ${wheel_z}" rpy="${wheel_r} ${wheel_p} ${wheel_ya}"/>
-        <mass value="5"/>
-        <cylinder_inertia m="5" r="${wheel_cylinder_radius}" h="${wheel_cylinder_height}"/>
+        <mass value="1"/>
+        <cylinder_inertia m="1" r="${wheel_cylinder_radius}" h="${wheel_cylinder_height}"/>
         <inertia
           ixx="1.0" ixy="0.0" ixz="0.0"

File: skyfood_ws/install/robot_description/share/robot_description/urdf/xacro_variables.xacro (robot description, xacro)
@@ -25,16 +25,19 @@
   <xacro:property name="chasis_box_ya" value="0" />
   <!--Chasis_caster-->
-  <xacro:property name="chasis_caster_x" value="-0.2" />
-  <xacro:property name="chasis_caster_y" value="0" />
-  <xacro:property name="chasis_caster_z" value="-0.047" />
   <xacro:property name="chasis_caster_r" value="0" />
   <xacro:property name="chasis_caster_p" value="0" />
   <xacro:property name="chasis_caster_ya" value="0" />
+  <xacro:property name="chasis_caster_x" value="-0.2" />
+  <xacro:property name="chasis_caster_y" value="0.145" />
+  <xacro:property name="chasis_caster_z" value="-0.047" />
   <xacro:property name="chasis_caster2_x" value="0.2" />
-  <xacro:property name="chasis_caster2_y" value="0" />
+  <xacro:property name="chasis_caster2_y" value="0.145" />
   <xacro:property name="chasis_caster2_z" value="-0.047" />
-  <xacro:property name="chasis_caster2_r" value="0" />
-  <xacro:property name="chasis_caster2_p" value="0" />
-  <xacro:property name="chasis_caster2_ya" value="0" />
+  <xacro:property name="chasis_caster3_x" value="-0.2" />
+  <xacro:property name="chasis_caster3_y" value="-0.145" />
+  <xacro:property name="chasis_caster3_z" value="-0.047" />
+  <xacro:property name="chasis_caster4_x" value="0.2" />
+  <xacro:property name="chasis_caster4_y" value="-0.145" />
+  <xacro:property name="chasis_caster4_z" value="-0.047" />
   <!--Wheel-->
   <xacro:property name="wheel_x" value="0" />

File: skyfood_ws/src/robot_description/urdf/robot_base.xacro (robot description, xacro)
@@ -13,7 +13,7 @@
     <pose>0 0 0.1 0 0 0</pose>
     <inertial>
-      <mass value="10.0"/>
+      <mass value="30.0"/>
       <origin xyz="0.0 0 0.1" rpy=" 0 0 0"/>
-      <box_inertia m="10" l="${chasis_box_length}" w="${chasis_box_width}" h="${chasis_box_height}"/>
+      <box_inertia m="30" l="${chasis_box_length}" w="${chasis_box_width}" h="${chasis_box_height}"/>
       <inertia
           ixx="0.5" ixy="0" ixz="0"
@@ -71,5 +71,5 @@
     </visual>
     <collision name='caster_collision2'>
-      <origin xyz="${chasis_caster2_x} ${chasis_caster2_y} ${chasis_caster2_z}" rpy=" ${chasis_caster2_r} ${chasis_caster2_p} ${chasis_caster2_ya}"/>
+      <origin xyz="${chasis_caster2_x} ${chasis_caster2_y} ${chasis_caster2_z}" rpy=" ${chasis_caster_r} ${chasis_caster_p} ${chasis_caster_ya}"/>
       <geometry>
         <sphere radius="${chasis_caster_radius}"/>
@@ -87,5 +87,51 @@
     </collision>
     <visual name='caster2_visual'>
-      <origin xyz="${chasis_caster2_x} ${chasis_caster2_y} ${chasis_caster2_z}" rpy=" ${chasis_caster2_r} ${chasis_caster2_p} ${chasis_caster2_ya}"/>
+      <origin xyz="${chasis_caster2_x} ${chasis_caster2_y} ${chasis_caster2_z}" rpy=" ${chasis_caster_r} ${chasis_caster_p} ${chasis_caster_ya}"/>
+      <geometry>
+        <sphere radius="${chasis_caster_radius}"/>
+      </geometry>
+      <material name="orange"/>
+    </visual>
+    <collision name='caster_collision3'>
+      <origin xyz="${chasis_caster3_x} ${chasis_caster3_y} ${chasis_caster3_z}" rpy=" ${chasis_caster_r} ${chasis_caster_p} ${chasis_caster_ya}"/>
+      <geometry>
+        <sphere radius="${chasis_caster_radius}"/>
+      </geometry>
+      <surface>
+        <friction>
+          <ode>
+            <mu>0</mu>
+            <mu2>0</mu2>
+            <slip1>1.0</slip1>
+            <slip2>1.0</slip2>
+          </ode>
+        </friction>
+      </surface>
+    </collision>
+    <visual name='caster3_visual'>
+      <origin xyz="${chasis_caster3_x} ${chasis_caster3_y} ${chasis_caster3_z}" rpy=" ${chasis_caster_r} ${chasis_caster_p} ${chasis_caster_ya}"/>
+      <geometry>
+        <sphere radius="${chasis_caster_radius}"/>
+      </geometry>
+      <material name="orange"/>
+    </visual>
+    <collision name='caster_collision4'>
+      <origin xyz="${chasis_caster4_x} ${chasis_caster4_y} ${chasis_caster4_z}" rpy=" ${chasis_caster_r} ${chasis_caster_p} ${chasis_caster_ya}"/>
+      <geometry>
+        <sphere radius="${chasis_caster_radius}"/>
+      </geometry>
+      <surface>
+        <friction>
+          <ode>
+            <mu>0</mu>
+            <mu2>0</mu2>
+            <slip1>1.0</slip1>
+            <slip2>1.0</slip2>
+          </ode>
+        </friction>
+      </surface>
+    </collision>
+    <visual name='caster4_visual'>
+      <origin xyz="${chasis_caster4_x} ${chasis_caster4_y} ${chasis_caster4_z}" rpy=" ${chasis_caster_r} ${chasis_caster_p} ${chasis_caster_ya}"/>
       <geometry>
         <sphere radius="${chasis_caster_radius}"/>
@@ -117,5 +163,5 @@
     <parent link="chassis"/>
     <child link="lidar_link"/>
-    <origin xyz="0 0 0.2" rpy="0 0 0"/>
+    <origin xyz="0 0 0.18" rpy="0 0 0"/>
   </joint>
   <link name="camera_link">
