Commit message: fix random stopping

File: skyfood_ws/install/robot_description/share/robot_description/urdf/wheels.xacro (robot description, xacro)
@@ -71,5 +71,5 @@
       <parent link="base_link"/>
       <axis xyz="0 1 0" rpy="0 0 0"/>
-      <dynamics damping="0.0" friction="0.01"/>
+      <dynamics damping="0.0" friction="0.0"/>
     </joint>
     <joint type="continuous" name="right_wheel_hinge">
@@ -78,5 +78,5 @@
       <parent link="base_link"/>
       <axis xyz="0 1 0" rpy="0 0 0"/>
-      <dynamics damping="0.0" friction="0.01"/>
+      <dynamics damping="0.0" friction="0.0"/>
     </joint>
   </xacro:macro>

File: skyfood_ws/src/robot_description/urdf/wheels.xacro (robot description, xacro)
@@ -71,5 +71,5 @@
       <parent link="base_link"/>
       <axis xyz="0 1 0" rpy="0 0 0"/>
-      <dynamics damping="0.5" friction="0.1"/>
+      <dynamics damping="0.0" friction="0.0"/>
     </joint>
     <joint type="continuous" name="right_wheel_hinge">
@@ -78,5 +78,5 @@
       <parent link="base_link"/>
       <axis xyz="0 1 0" rpy="0 0 0"/>
-      <dynamics damping="0.5" friction="0.1"/>
+      <dynamics damping="0.0" friction="0.0"/>
     </joint>
   </xacro:macro>
