Commit message: depth cameras xacros

File: skyfood_ws/install/robot_description/share/robot_description/urdf/robot_base.xacro (robot description, xacro)
@@ -176,4 +176,31 @@
     <origin xyz="0.239 0 0.84" rpy="0 0 0"/>
   </joint>
+  <link name="camera_link_optical">
+  </link>
+  <joint name="camera_optical_joint" type="fixed">
+    <parent link="camera_link"/>
+    <child link="camera_link_optical"/>
+    <origin xyz="0 0 0" rpy="-1.5707 0 -1.5707"/>
+  </joint>
+  <link name="camera_link_2">
+    <visual name="camera_visual_2">
+      <origin xyz="0 0 0" rpy="0 0 0"/>
+      <geometry>
+        <box size="0.02 0.15 0.1"/>
+      </geometry>
+    </visual>
+  </link>
+  <joint name="camera_joint_2" type="fixed">
+    <parent link="chassis"/>
+    <child link="camera_link_2"/>
+    <origin xyz="0.239 0 0.79" rpy="0 0.523598 0"/>
+  </joint>
+  <link name="camera_link_optical_2">
+  </link>
+  <joint name="camera_optical_joint_2" type="fixed">
+    <parent link="camera_link_2"/>
+    <child link="camera_link_optical_2"/>
+    <origin xyz="0 0 0" rpy="-1.5707 0 -1.5707"/>
+  </joint>
   <!-- Include wheel macro -->
   <xacro:wheels_macro />

File: skyfood_ws/install/robot_description/share/robot_description/urdf/sensors.xacro (robot description, xacro)
@@ -49,26 +49,51 @@
         </sensor>
     </gazebo>
-    <!-- Camera Plugin -->
+    <!-- Depth Camera Plugin -->
     <gazebo reference="camera_link">
-        <sensor name="camera" type="camera">
+        <sensor name="camera" type="depth">
             <pose>0.11 0 0 0 0 0</pose>
             <visualize>true</visualize>
             <update_rate>10</update_rate>
-            <image_topic_name>camera/image_raw</image_topic_name>
-            <camera_info_topic_name>camera/camera_info</camera_info_topic_name>
             <camera>
-                <horizontal_fov>1.089</horizontal_fov>
+                <horizontal_fov>1.3439</horizontal_fov>
                 <image>
-                    <format>R8G8B8</format>
+                    <format>B8G8R8</format>
                     <width>640</width>
-                    <height>480</height>
+                    <height>400</height>
                 </image>
                 <clip>
-                    <near>0.05</near>
-                    <far>8.0</far>
+                    <near>0.1</near>
+                    <far>100.0</far>
                 </clip>
             </camera>
             <plugin name="camera_controller" filename="libgazebo_ros_camera.so">
-                <frame_name>camera_link</frame_name>
+                <frame_name>camera_link_optical</frame_name>
+                <min_depth>0.7</min_depth>
+                <max_depth>12.0</max_depth>
+            </plugin>
+        </sensor>
+    </gazebo>
+    <!-- Second Depth Camera Plugin -->
+    <gazebo reference="camera_link_2">
+        <sensor name="camera_2" type="depth">
+            <pose>0.11 0 0 0 0 0</pose>
+            <visualize>true</visualize>
+            <update_rate>10</update_rate>
+            <camera>
+                <horizontal_fov>1.25664</horizontal_fov>
+                <image>
+                    <format>B8G8R8</format>
+                    <width>320</width>
+                    <height>240</height>
+                </image>
+                <clip>
+                    <near>0.15</near>
+                    <far>1.5</far>
+                </clip>
+            </camera>
+            <plugin name="camera_controller_2" filename="libgazebo_ros_camera.so">
+                <frame_name>camera_link_optical_2</frame_name>
+                <min_depth>0.15</min_depth>
+                <max_depth>1.5</max_depth>
             </plugin>
         </sensor>
