Commit message: fix swapped wheel coordinates

File: skyfood_ws/install/robot_description/share/robot_description/urdf/sensors.xacro (robot description, xacro)
@@ -102,9 +102,9 @@
     <gazebo>
         <plugin name="gazebo_ros_diff_drive" filename="libgazebo_ros_diff_drive.so">
-            <update_rate>10</update_rate>
+            <update_rate>50</update_rate>
             <left_joint>left_wheel_hinge</left_joint>
             <right_joint>right_wheel_hinge</right_joint>
-            <wheel_separation>0.4</wheel_separation>
-            <wheel_diameter>0.2</wheel_diameter>
+            <wheel_separation>0.332</wheel_separation>
+            <wheel_diameter>0.17</wheel_diameter>
             <command_topic>cmd_vel</command_topic>
             <publish_odom>true</publish_odom>

File: skyfood_ws/install/robot_description/share/robot_description/urdf/xacro_variables.xacro (robot description, xacro)
@@ -49,8 +49,8 @@
 <!--Joint variables-->
   <xacro:property name="right_wheel_x" value="0.0" />
-  <xacro:property name="right_wheel_y" value="0.166" />
+  <xacro:property name="right_wheel_y" value="-0.166" />
   <xacro:property name="right_wheel_z" value="0" />
   <xacro:property name="left_wheel_x" value="0" />
-  <xacro:property name="left_wheel_y" value="-0.166" />
+  <xacro:property name="left_wheel_y" value="0.166" />
   <xacro:property name="left_wheel_z" value="0" />
 </robot>
