Commit message: fix wobble

File: skyfood_ws/src/robot_description/urdf/caster_ball.xacro (robot description, xacro)
@@ -48,50 +48,50 @@
       <material name="orange"/>
     </visual>
+    <collision name='caster_collision3'>
+      <origin xyz="${chasis_caster3_x} ${chasis_caster3_y} ${chasis_caster3_z}" rpy=" ${chasis_caster_r} ${chasis_caster_p} ${chasis_caster_ya}"/>
+      <geometry>
+        <sphere radius="${chasis_caster_radius}"/>
+      </geometry>
+      <surface>
+        <friction>
+          <ode>
+            <mu>0</mu>
+            <mu2>0</mu2>
+            <slip1>1.0</slip1>
+            <slip2>1.0</slip2>
+          </ode>
+        </friction>
+      </surface>
+    </collision>
+    <visual name='caster3_visual'>
+      <origin xyz="${chasis_caster3_x} ${chasis_caster3_y} ${chasis_caster3_z}" rpy=" ${chasis_caster_r} ${chasis_caster_p} ${chasis_caster_ya}"/>
+      <geometry>
+        <sphere radius="${chasis_caster_radius}"/>
+      </geometry>
+      <material name="orange"/>
+    </visual>
+    <collision name='caster_collision4'>
+      <origin xyz="${chasis_caster4_x} ${chasis_caster4_y} ${chasis_caster4_z}" rpy=" ${chasis_caster_r} ${chasis_caster_p} ${chasis_caster_ya}"/>
+      <geometry>
+        <sphere radius="${chasis_caster_radius}"/>
+      </geometry>
+      <surface>
+        <friction>
+          <ode>
+            <mu>0</mu>
+            <mu2>0</mu2>
+            <slip1>1.0</slip1>
+            <slip2>1.0</slip2>
+          </ode>
+        </friction>
+      </surface>
+    </collision>
+    <visual name='caster4_visual'>
+      <origin xyz="${chasis_caster4_x} ${chasis_caster4_y} ${chasis_caster4_z}" rpy=" ${chasis_caster_r} ${chasis_caster_p} ${chasis_caster_ya}"/>
+      <geometry>
+        <sphere radius="${chasis_caster_radius}"/>
+      </geometry>
+      <material name="orange"/>
+    </visual>
   </xacro:macro>
-  <collision name='caster_collision3'>
-    <origin xyz="${chasis_caster3_x} ${chasis_caster3_y} ${chasis_caster3_z}" rpy=" ${chasis_caster_r} ${chasis_caster_p} ${chasis_caster_ya}"/>
-    <geometry>
-      <sphere radius="${chasis_caster_radius}"/>
-    </geometry>
-    <surface>
-      <friction>
-        <ode>
-          <mu>0</mu>
-          <mu2>0</mu2>
-          <slip1>1.0</slip1>
-          <slip2>1.0</slip2>
-        </ode>
-      </friction>
-    </surface>
-  </collision>
-  <visual name='caster3_visual'>
-    <origin xyz="${chasis_caster3_x} ${chasis_caster3_y} ${chasis_caster3_z}" rpy=" ${chasis_caster_r} ${chasis_caster_p} ${chasis_caster_ya}"/>
-    <geometry>
-      <sphere radius="${chasis_caster_radius}"/>
-    </geometry>
-    <material name="orange"/>
-  </visual>
-  <collision name='caster_collision4'>
-    <origin xyz="${chasis_caster4_x} ${chasis_caster4_y} ${chasis_caster4_z}" rpy=" ${chasis_caster_r} ${chasis_caster_p} ${chasis_caster_ya}"/>
-    <geometry>
-      <sphere radius="${chasis_caster_radius}"/>
-    </geometry>
-    <surface>
-      <friction>
-        <ode>
-          <mu>0</mu>
-          <mu2>0</mu2>
-          <slip1>1.0</slip1>
-          <slip2>1.0</slip2>
-        </ode>
-      </friction>
-    </surface>
-  </collision>
-  <visual name='caster4_visual'>
-    <origin xyz="${chasis_caster4_x} ${chasis_caster4_y} ${chasis_caster4_z}" rpy=" ${chasis_caster_r} ${chasis_caster_p} ${chasis_caster_ya}"/>
-    <geometry>
-      <sphere radius="${chasis_caster_radius}"/>
-    </geometry>
-    <material name="orange"/>
-  </visual>
 </robot>

File: skyfood_ws/src/robot_description/urdf/robot_base.xacro (robot description, xacro)
@@ -13,11 +13,16 @@
     <pose>0 0 0.1 0 0 0</pose>
     <inertial>
+      <!-- Combined CoM: base at z=0, tower (0.64m tall) centered at z=0.58m
+           Approximate CoM ≈ z=0.35m relative to chassis link origin -->
+      <origin xyz="0.0 0 0.35" rpy="0 0 0"/>
       <mass value="30.0"/>
-      <origin xyz="0.0 0 0.1" rpy=" 0 0 0"/>
-      <box_inertia m="30" l="${chasis_box_length}" w="${chasis_box_width}" h="${chasis_box_height}"/>
+      <!-- Ixx = (1/12)*m*(w^2+h^2) using tower dims as dominant: w=0.448, H=0.64 -->
+      <!-- Approximate as tall box: Ixx ~= (1/12)*30*(0.448^2 + 0.64^2) = 1.523 -->
+      <!-- Iyy ~= (1/12)*30*(0.478^2 + 0.64^2) = 1.597                          -->
+      <!-- Izz ~= (1/12)*30*(0.478^2 + 0.448^2) = 0.803                          -->
       <inertia
-          ixx="0.5" ixy="0" ixz="0"
-          iyy="1.0" iyz="0"
-          izz="0.1"
+          ixx="1.52" ixy="0" ixz="0"
+          iyy="1.60" iyz="0"
+          izz="0.80"
       />
     </inertial>
@@ -46,96 +51,4 @@
       </geometry>
       <material name="red"/>
-    </visual>
-    <collision name='caster_collision'>
-      <origin xyz="${chasis_caster_x} ${chasis_caster_y} ${chasis_caster_z}" rpy=" ${chasis_caster_r} ${chasis_caster_p} ${chasis_caster_ya}"/>
-      <geometry>
-        <sphere radius="${chasis_caster_radius}"/>
-      </geometry>
-      <surface>
-        <friction>
-          <ode>
-            <mu>0</mu>
-            <mu2>0</mu2>
-            <slip1>1.0</slip1>
-            <slip2>1.0</slip2>
-          </ode>
-        </friction>
-      </surface>
-    </collision>
-    <visual name='caster_visual'>
-      <origin xyz="${chasis_caster_x} ${chasis_caster_y} ${chasis_caster_z}" rpy=" ${chasis_caster_r} ${chasis_caster_p} ${chasis_caster_ya}"/>
-      <geometry>
-        <sphere radius="${chasis_caster_radius}"/>
-      </geometry>
-      <material name="orange"/>
-    </visual>
-    <collision name='caster_collision2'>
-      <origin xyz="${chasis_caster2_x} ${chasis_caster2_y} ${chasis_caster2_z}" rpy=" ${chasis_caster_r} ${chasis_caster_p} ${chasis_caster_ya}"/>
-      <geometry>
-        <sphere radius="${chasis_caster_radius}"/>
-      </geometry>
-      <surface>
-        <friction>
-          <ode>
-            <mu>0</mu>
-            <mu2>0</mu2>
-            <slip1>1.0</slip1>
-            <slip2>1.0</slip2>
-          </ode>
-        </friction>
-      </surface>
-    </collision>
-    <visual name='caster2_visual'>
-      <origin xyz="${chasis_caster2_x} ${chasis_caster2_y} ${chasis_caster2_z}" rpy=" ${chasis_caster_r} ${chasis_caster_p} ${chasis_caster_ya}"/>
-      <geometry>
-        <sphere radius="${chasis_caster_radius}"/>
-      </geometry>
-      <material name="orange"/>
-    </visual>
-    <collision name='caster_collision3'>
-      <origin xyz="${chasis_caster3_x} ${chasis_caster3_y} ${chasis_caster3_z}" rpy=" ${chasis_caster_r} ${chasis_caster_p} ${chasis_caster_ya}"/>
-      <geometry>
-        <sphere radius="${chasis_caster_radius}"/>
-      </geometry>
-      <surface>
-        <friction>
-          <ode>
-            <mu>0</mu>
-            <mu2>0</mu2>
-            <slip1>1.0</slip1>
-            <slip2>1.0</slip2>
-          </ode>
-        </friction>
-      </surface>
-    </collision>
-    <visual name='caster3_visual'>
-      <origin xyz="${chasis_caster3_x} ${chasis_caster3_y} ${chasis_caster3_z}" rpy=" ${chasis_caster_r} ${chasis_caster_p} ${chasis_caster_ya}"/>
-      <geometry>
-        <sphere radius="${chasis_caster_radius}"/>
-      </geometry>
-      <material name="orange"/>
-    </visual>
-    <collision name='caster_collision4'>
-      <origin xyz="${chasis_caster4_x} ${chasis_caster4_y} ${chasis_caster4_z}" rpy=" ${chasis_caster_r} ${chasis_caster_p} ${chasis_caster_ya}"/>
-      <geometry>
-        <sphere radius="${chasis_caster_radius}"/>
-      </geometry>
-      <surface>
-        <friction>
-          <ode>
-            <mu>0</mu>
-            <mu2>0</mu2>
-            <slip1>1.0</slip1>
-            <slip2>1.0</slip2>
-          </ode>
-        </friction>
-      </surface>
-    </collision>
-    <visual name='caster4_visual'>
-      <origin xyz="${chasis_caster4_x} ${chasis_caster4_y} ${chasis_caster4_z}" rpy=" ${chasis_caster_r} ${chasis_caster_p} ${chasis_caster_ya}"/>
-      <geometry>
-        <sphere radius="${chasis_caster_radius}"/>
-      </geometry>
-      <material name="orange"/>
     </visual>
   </link>

File: skyfood_ws/src/robot_description/urdf/wheels.xacro (robot description, xacro)
@@ -27,9 +27,11 @@
         <origin xyz="${wheel_x} ${wheel_y} ${wheel_z}" rpy="${wheel_r} ${wheel_p} ${wheel_ya}"/>
         <mass value="1"/>
-        <cylinder_inertia m="1" r="${wheel_cylinder_radius}" h="${wheel_cylinder_height}"/>
+        <!-- Cylinder inertia: r=0.085, h=0.045, m=1
+             Ixx = Iyy = (1/12)*m*(3r^2+h^2) = (1/12)*(3*0.007225+0.002025) = 0.001972
+             Izz = (1/2)*m*r^2 = 0.5*0.007225 = 0.003613 -->
         <inertia
-          ixx="1.0" ixy="0.0" ixz="0.0"
-          iyy="1.0" iyz="0.0"
-          izz="1.0"/>
+          ixx="0.00197" ixy="0.0" ixz="0.0"
+          iyy="0.00197" iyz="0.0"
+          izz="0.00361"/>
       </inertial>
     </link>
@@ -59,9 +61,11 @@
         <origin xyz="${wheel_x} ${wheel_y} ${wheel_z}" rpy="${wheel_r} ${wheel_p} ${wheel_ya}"/>
         <mass value="1"/>
-        <cylinder_inertia m="1" r="${wheel_cylinder_radius}" h="${wheel_cylinder_height}"/>
+        <!-- Cylinder inertia: r=0.085, h=0.045, m=1
+             Ixx = Iyy = (1/12)*m*(3r^2+h^2) = 0.001972
+             Izz = (1/2)*m*r^2 = 0.003613 -->
         <inertia
-          ixx="1.0" ixy="0.0" ixz="0.0"
-          iyy="1.0" iyz="0.0"
-          izz="1.0"/>
+          ixx="0.00197" ixy="0.0" ixz="0.0"
+          iyy="0.00197" iyz="0.0"
+          izz="0.00361"/>
       </inertial>
     </link>
@@ -71,5 +75,5 @@
       <parent link="base_link"/>
       <axis xyz="0 1 0" rpy="0 0 0"/>
-      <joint_properties damping="0.0" friction="0.0"/>
+      <dynamics damping="0.5" friction="0.1"/>
     </joint>
     <joint type="continuous" name="right_wheel_hinge">
@@ -78,5 +82,5 @@
       <parent link="base_link"/>
       <axis xyz="0 1 0" rpy="0 0 0"/>
-      <joint_properties damping="0.0" friction="0.0"/>
+      <dynamics damping="0.5" friction="0.1"/>
     </joint>
   </xacro:macro>
